Commit message: Починил inverse_kinematic

File: description.urdf (robot description, URDF)
Before this commit: robot myfirst, 7 links, 6 joints
Joints:
- joint joint_J0: limit lower=0.0 upper=6.28319 effort=0.0 velocity=0.0 -> lower=-1.57 upper=1.57 effort=0.0 velocity=0.0
- joint joint_J1: limit lower=0.6108 upper=1.13446 effort=0.0 velocity=0.0 -> lower=0.5236 upper=0.9599 effort=0.0 velocity=0.0
- joint joint_J2: limit lower=0.95993 upper=1.5708 effort=0.0 velocity=0.0 -> lower=1.1345 upper=1.8326 effort=0.0 velocity=0.0
- joint joint_J3: limit lower=0.0 upper=4.7123 effort=0.0 velocity=0.0 -> lower=-3.14 upper=0.0 effort=0.0 velocity=0.0
- joint joint_J4: limit lower=0.0 upper=3.14159 effort=0.0 velocity=0.0 -> lower=-1.57 upper=1.57 effort=0.0 velocity=0.0
- joint joint_J5: limit lower=0.0 upper=4.71239 effort=0.0 velocity=0.0 -> lower=0.0 upper=3.1416 effort=0.0 velocity=0.0

Commit message: Исправлен urdf

File: description.urdf (robot description, URDF)
Before this commit: robot myfirst, 7 links, 6 joints
Links:
- added link TOOL; visual cylinder length=0.007 radius=0.045
- link J0: geometry visual box size=0.1 0.1 0.1
Joints:
- added joint TOOL_joint: type fixed, parent J5, child TOOL, origin xyz=0.0 0.0 0.11 rpy=0.0 0.0 0.0
- joint joint_J0: origin (none) -> xyz=0.0 0.0 0.0
- joint joint_J1: limit lower=0.5236 upper=0.9599 effort=0.0 velocity=0.0 -> lower=0.0 upper=0.6109 effort=0.0 velocity=0.0; origin xyz=0.065 0.0 0.055 rpy=1.5707 0.0 0.0 -> xyz=0.07 0.0 0.0 rpy=1.57 -0.4363 0.0
- joint joint_J2: limit lower=1.1345 upper=1.8326 effort=0.0 velocity=0.0 -> lower=0.0 upper=0.6109 effort=0.0 velocity=0.0; origin xyz=0.0 0.42 0.0 rpy=0.0 0.0 0.0 -> xyz=0.0 0.425 0.0 rpy=0.0 0.0 1.2217
- joint joint_J3: origin xyz=0.0 0.44 0.0 rpy=1.57 0.0 -0.174533 -> xyz=0.0 0.445 0.0 rpy=1.57 0.0 -0.174533
- joint joint_J5: origin xyz=0.0 0.087 0.0 rpy=-1.5708 0.0 0.0 -> xyz=0.0 0.09 0.0 rpy=-1.5708 0.0 0.0
